File: pcb/videogame.kicad_sch (KiCad schematic)
At the start: 0 parts

Commit message: feat: scheme completed
Parts:
- added A1: RaspberryPi_Pico, Module:RaspberryPi_Pico_Common_Unspecified, symbol MCU_Module:RaspberryPi_Pico
- added BT1: Battery_Cell, Package_SON:Texas_DRC0010J_ThermalVias, symbol Device:Battery_Cell
- added BZ1: Buzzer, symbol Device:Buzzer
- added DS1: (no value), symbol CONSOLE_LIB:st7789_8p_1spi
- added J1: Micro_SD_Card, Package_DFN_QFN:QFN-48-1EP_7x7mm_P0.5mm_EP5.15x5.15mm, symbol Connector:Micro_SD_Card
- added J2: Conn_01x04, Connector_RJ:RJ45_Abracon_ARJP11A-MA_Horizontal, symbol Connector_Generic:Conn_01x04
- added SW1, SW2, SW3, SW4, SW5, SW6, SW7, SW8: SW_Push, PCM_marbastlib-he:SW_MX_HE_0deg_1u, symbol Switch:SW_Push
- added SW9: SW_SPDT, Button_Switch_THT:SW_NKK_GW12LJP, symbol Switch:SW_SPDT
Connections:
- new net +3V3: A1.36 (3V3), DS1.1 (LEDA), DS1.7 (VDD), J1.4 (VDD)
- new net BAT+: BT1.1 (+), J2.1 (Pin_1)
- new net BUTTON_A: A1.9 (GPIO6), SW2.1
- new net BUTTON_B: A1.10 (GPIO7), SW4.1
- new net BUTTON_DOWN: A1.5 (GPIO3), SW5.1
- new net BUTTON_LEFT: A1.6 (GPIO4), SW6.1
- new net BUTTON_RIGHT: A1.7 (GPIO5), SW7.1
- new net BUTTON_SELECT: A1.12 (GPIO9), SW1.1
- new net BUTTON_START: A1.11 (GPIO8), SW3.1
- new net BUTTON_UP: A1.4 (GPIO2), SW8.1
- new net BUZZER+: BZ1.1 (+)
- new net CS: A1.17 (GPIO13), DS1.8 (CS)
- new net D_C: A1.19 (GPIO14), DS1.4 (D/C)
- new net GND: A1.13 (GND), A1.18 (GND), A1.23 (GND), A1.28 (GND), A1.3 (GND), A1.38 (GND), A1.8 (GND), BT1.2 (-), BZ1.2 (-), DS1.2 (GND), DS1.S1 (GND), DS1.S2 (GND), J1.6 (VSS), J1.SH (SHIELD), J2.2 (Pin_2), J2.4 (Pin_4), SW1.2, SW2.2, SW3.2, SW4.2, SW5.2, SW6.2, SW7.2, SW8.2
- new net OUT+: J2.3 (Pin_3), SW9.1 (A)
- new net RESET: A1.20 (GPIO15), DS1.3 (RESET)
- new net SCL: A1.14 (GPIO10), DS1.6 (SCL)
- new net SDA: A1.15 (GPIO11), DS1.5 (SDA)
- new net SD_CS: A1.21 (GPIO16), J1.2 (DAT3/CD)
- new net SD_MISO: A1.22 (GPIO17), J1.7 (DAT0)
- new net SD_MOSI: A1.25 (GPIO19), J1.3 (CMD)
- new net SD_SCK: A1.24 (GPIO18), J1.5 (CLK)
- new net SW_VS: A1.39 (VSYS), SW9.2 (B)
- no-connect marks 0 -> 17
Other:
- note added: "BUTTONs"
- note added: "Battery Cell"
- note added: "Buzzer"
- note added: "MODULE USB-C TP4056"
- note added: "Micro SD Card"
- note added: "Microcontroladora"
- note added: "OLED Display"
- note added: "ON/OFF Switch"
